File: templates/2-layer/000002 XXX Rev 1.00.sch (EAGLE design)
At the start: 20 parts, among them X1 PAD_TEST_GROUND_HOOK

Commit message: 2-layer template
Parts:
- added ART2: ART_SN_LABEL-08X24, Custom_Eagle_KD:ART_SN_LABEL-08X24
Other:
- moved on the sheet: ART1, LOGO2, LOGO3, MTG5, MTG6
Changed lines of the file:
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@@
 <?xml version="1.0" encoding="utf-8"?>
 <!DOCTYPE eagle SYSTEM "eagle.dtd">
-<eagle version="9.4.2">
+<eagle version="9.6.2">
 <drawing>
 <settings>
@@
 <layers>
 <layer number="1" name="Top" color="4" fill="1" visible="no" active="no"/>
+<layer number="2" name="Route2" color="1" fill="3" visible="no" active="no"/>
+<layer number="3" name="Route3" color="4" fill="3" visible="no" active="no"/>
+<layer number="4" name="Route4" color="1" fill="4" visible="no" active="no"/>
+<layer number="5" name="Route5" color="4" fill="4" visible="no" active="no"/>
+<layer number="6" name="Route6" color="1" fill="8" visible="no" active="no"/>
+<layer number="7" name="Route7" color="4" fill="8" visible="no" active="no"/>
+<layer number="8" name="Route8" color="1" fill="2" visible="no" active="no"/>
+<layer number="9" name="Route9" color="4" fill="2" visible="no" active="no"/>
+<layer number="10" name="Route10" color="1" fill="7" visible="no" active="no"/>
+<layer number="11" name="Route11" color="4" fill="7" visible="no" active="no"/>
+<layer number="12" name="Route12" color="1" fill="5" visible="no" active="no"/>
+<layer number="13" name="Route13" color="4" fill="5" visible="no" active="no"/>
+<layer number="14" name="Route14" color="1" fill="6" visible="no" active="no"/>
+<layer number="15" name="Route15" color="4" fill="6" visible="no" active="no"/>
 <layer number="16" name="Bottom" color="1" fill="1" visible="no" active="no"/>
 <layer number="17" name="Pads" color="2" fill="1" visible="no" active="no"/>
@@
 <part name="FRAME9" library="Custom_Eagle_KD" deviceset="ART_FRAME_A3" device=""/>
 <part name="FRAME10" library="Custom_Eagle_KD" deviceset="ART_FRAME_A3" device=""/>
+<part name="ART2" library="Custom_Eagle_KD" deviceset="ART_SN_LABEL" device="-08X24"/>
 </parts>
 <sheets>
@@
 <text x="515.62" y="452.12" size="2.54" layer="97">Fiducials</text>
 <wire x1="607.06" y1="444.5" x2="513.08" y2="444.5" width="0.1524" layer="97" style="longdash"/>
-<wire x1="513.08" y1="444.5" x2="513.08" y2="401.32" width="0.1524" layer="97" style="longdash"/>
-<wire x1="513.08" y1="401.32" x2="607.06" y2="401.32" width="0.1524" layer="97" style="longdash"/>
-<wire x1="607.06" y1="401.32" x2="607.06" y2="444.5" width="0.1524" layer="97" style="longdash"/>
-<text x="515.62" y="403.86" size="2.54" layer="97">Artwork</text>
-<wire x1="607.06" y1="396.24" x2="513.08" y2="396.24" width="0.1524" layer="97" style="longdash"/>
-<wire x1="513.08" y1="396.24" x2="513.08" y2="347.98" width="0.1524" layer="97" style="longdash"/>
+<wire x1="513.08" y1="444.5" x2="513.08" y2="383.54" width="0.1524" layer="97" style="longdash"/>
+<wire x1="513.08" y1="383.54" x2="607.06" y2="383.54" width="0.1524" layer="97" style="longdash"/>
+<wire x1="607.06" y1="383.54" x2="607.06" y2="444.5" width="0.1524" layer="97" style="longdash"/>
+<text x="515.62" y="386.08" size="2.54" layer="97">Artwork</text>
+<wire x1="607.06" y1="381" x2="513.08" y2="381" width="0.1524" layer="97" style="longdash"/>
+<wire x1="513.08" y1="381" x2="513.08" y2="347.98" width="0.1524" layer="97" style="longdash"/>
 <wire x1="513.08" y1="347.98" x2="607.06" y2="347.98" width="0.1524" layer="97" style="longdash"/>
-<wire x1="607.06" y1="347.98" x2="607.06" y2="396.24" width="0.1524" layer="97" style="longdash"/>
+<wire x1="607.06" y1="347.98" x2="607.06" y2="381" width="0.1524" layer="97" style="longdash"/>
 <text x="515.62" y="350.52" size="2.54" layer="97">Tester alignment holes</text>
 <wire x1="706.12" y1="497.84" x2="612.14" y2="497.84" width="0.1524" layer="97" style="longdash"/>
@@
 <attribute name="NAME" x="579.12" y="473.202" size="1.778" layer="95" align="bottom-center"/>
 </instance>
-<instance part="LOGO2" gate="G$1" x="558.8" y="424.18" smashed="yes">
-<attribute name="CODE" x="558.8" y="424.18" size="1.778" layer="96" align="center"/>
-<attribute name="NAME" x="558.8" y="420.624" size="1.778" layer="95" align="top-center"/>
-</instance>
-<instance part="LOGO3" gate="G$1" x="558.8" y="414.02" smashed="yes">
-<attribute name="CODE" x="558.8" y="414.02" size="1.778" layer="96" align="center"/>
-<attribute name="NAME" x="558.8" y="410.464" size="1.778" layer="95" align="top-center"/>
-</instance>
-<instance part="MTG5" gate="G$1" x="546.1" y="368.3" smashed="yes">
-<attribute name="NAME" x="546.1" y="372.872" size="1.778" layer="95" align="bottom-center"/>
-<attribute name="CODE" x="546.1" y="372.364" size="1.27" layer="96" align="top-center"/>
-</instance>
-<instance part="MTG6" gate="G$1" x="546.1" y="378.46" smashed="yes">
-<attribute name="NAME" x="546.1" y="383.032" size="1.778" layer="95" align="bottom-center"/>
-<attribute name="CODE" x="546.1" y="382.524" size="1.27" layer="96" align="top-center"/>
+<instance part="LOGO2" gate="G$1" x="561.34" y="421.64" smashed="yes">
+<attribute name="CODE" x="561.34" y="421.64" size="1.778" layer="96" align="center"/>
+<attribute name="NAME" x="561.34" y="418.084" size="1.778" layer="95" align="top-center"/>
+</instance>
+<instance part="LOGO3" gate="G$1" x="561.34" y="411.48" smashed="yes">
+<attribute name="CODE" x="561.34" y="411.48" size="1.778" layer="96" align="center"/>
+<attribute name="NAME" x="561.34" y="407.924" size="1.778" layer="95" align="top-center"/>
+</instance>
+<instance part="MTG5" gate="G$1" x="543.56" y="365.76" smashed="yes">
+<attribute name="NAME" x="543.56" y="370.332" size="1.778" layer="95" align="bottom-center"/>
+<attribute name="CODE" x="543.56" y="369.824" size="1.27" layer="96" align="top-center"/>
+</instance>
+<instance part="MTG6" gate="G$1" x="574.04" y="365.76" smashed="yes">
+<attribute name="NAME" x="574.04" y="370.332" size="1.778" layer="95" align="bottom-center"/>
+<attribute name="CODE" x="574.04" y="369.824" size="1.27" layer="96" align="top-center"/>
 </instance>
 <instance part="MTG4" gate="G$1" x="642.62" y="459.74" smashed="yes">
@@
 <attribute name="CODE" x="673.1" y="448.564" size="1.27" layer="96" align="top-center"/>
 </instance>
-<instance part="ART1" gate="G$1" x="558.8" y="434.34" smashed="yes">
-<attribute name="CODE" x="558.8" y="434.34" size="1.778" layer="96" align="center"/>
-<attribute name="NAME" x="558.8" y="430.784" size="1.778" layer="95" align="top-center"/>
+<instance part="ART1" gate="G$1" x="561.34" y="431.8" smashed="yes">
+<attribute name="CODE" x="561.34" y="431.8" size="1.778" layer="96" align="center"/>
+<attribute name="NAME" x="561.34" y="428.244" size="1.778" layer="95" align="top-center"/>
 </instance>
 <instance part="TP1" gate="*" x="165.1" y="1000.76" smashed="yes">
@@
 <attribute name="PCBA_PN" x="770.89" y="11.43" size="2.54" layer="94" align="center"/>
 </instance>
+<instance part="ART2" gate="G$1" x="561.34" y="401.32" smashed="yes">
+<attribute name="CODE" x="561.34" y="401.32" size="1.778" layer="96" align="center"/>
+<attribute name="NAME" x="561.34" y="397.764" size="1.778" layer="95" align="top-center"/>
+</instance>
 </instances>

Commit message: Changed templates to managed libraries
Parts:
- MTG5, MTG6: value HOL_3.2/6.0_NP -> HOL_3.2/6.0_NP-NOSILK; device Custom_Eagle_KD:HOL_3.2/6.0_NP -> Custom_Eagle_KD:HOL_3.2/6.0_NP-NOSILK
Changed lines of the file:
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@@
 </classes>
 <parts>
-<part name="SHEETINFO1" library="Custom_Eagle_KD" deviceset="ART_SHEET_INFO_1-16" device=""/>
-<part name="TEST_POINTS1" library="Custom_Eagle_KD" deviceset="ART_TEST_POINTS" device=""/>
-<part name="FIDUCIAL1" library="Custom_Eagle_KD" deviceset="FIDUCIAL" device=""/>
-<part name="FIDUCIAL2" library="Custom_Eagle_KD" deviceset="FIDUCIAL" device=""/>
-<part name="FIDUCIAL3" library="Custom_Eagle_KD" deviceset="FIDUCIAL" device=""/>
-<part name="FIDUCIAL4" library="Custom_Eagle_KD" deviceset="FIDUCIAL" device=""/>
-<part name="FIDUCIAL5" library="Custom_Eagle_KD" deviceset="FIDUCIAL" device=""/>
-<part name="FIDUCIAL6" library="Custom_Eagle_KD" deviceset="FIDUCIAL" device=""/>
-<part name="LOGO2" library="Custom_Eagle_KD" deviceset="ART_LOGO_TEXT_2.5MM" device="-SILK"/>
-<part name="LOGO3" library="Custom_Eagle_KD" deviceset="ART_LOGO_TEXT_2.5MM" device="-MASK"/>
-<part name="MTG5" library="Custom_Eagle_KD" deviceset="HOL_3.2/6.0_NP" device=""/>
-<part name="MTG6" library="Custom_Eagle_KD" deviceset="HOL_3.2/6.0_NP" device=""/>
-<part name="MTG4" library="Custom_Eagle_KD" deviceset="HOL_3.2/6.0_PTH" device="-3.2/6.0_PTH"/>
-<part name="GND18" library="Custom_Supply_Symbols_KD" deviceset="GND" device=""/>
-<part name="GND16" library="Custom_Supply_Symbols_KD" deviceset="GND" device=""/>
-<part name="REVINFO1" library="Custom_Eagle_KD" deviceset="ART_REVISION_HISTORY" device=""/>
-<part name="X1" library="Custom_Eagle_KD" deviceset="PAD_TEST_GROUND_HOOK" device=""/>
-<part name="MTG1" library="Custom_Eagle_KD" deviceset="HOL_2.2/4.2_NP" device=""/>
-<part name="MTG2" library="Custom_Eagle_KD" deviceset="HOL_2.2/4.2_NP" device=""/>
-<part name="MTG3" library="Custom_Eagle_KD" deviceset="HOL_2.2/4.2_NP" device=""/>
-<part name="MTG7" library="Custom_Eagle_KD" deviceset="HOL_2.2/4.2_NP" device=""/>
-<part name="ART1" library="Custom_Eagle_KD" deviceset="ART_QC" device=""/>
-<part name="TP1" library="Custom_Eagle_KD" deviceset="PAD_TEST_POINT" device="-2.5MM"/>
-<part name="TP2" library="Custom_Eagle_KD" deviceset="PAD_TEST_POINT" device="-2.5MM"/>
-<part name="TP3" library="Custom_Eagle_KD" deviceset="PAD_TEST_POINT" device="-2.5MM"/>
-<part name="FRAME1" library="Custom_Eagle_KD" deviceset="ART_FRAME_A3" device=""/>
-<part name="FRAME2" library="Custom_Eagle_KD" deviceset="ART_FRAME_A3" device=""/>
-<part name="FRAME3" library="Custom_Eagle_KD" deviceset="ART_FRAME_A3" device=""/>
-<part name="FRAME4" library="Custom_Eagle_KD" deviceset="ART_FRAME_A3" device=""/>
-<part name="FRAME5" library="Custom_Eagle_KD" deviceset="ART_FRAME_A3" device=""/>
-<part name="FRAME6" library="Custom_Eagle_KD" deviceset="ART_FRAME_A3" device=""/>
-<part name="FRAME7" library="Custom_Eagle_KD" deviceset="ART_FRAME_A3" device=""/>
-<part name="FRAME8" library="Custom_Eagle_KD" deviceset="ART_FRAME_A3" device=""/>
-<part name="FRAME9" library="Custom_Eagle_KD" deviceset="ART_FRAME_A3" device=""/>
-<part name="FRAME10" library="Custom_Eagle_KD" deviceset="ART_FRAME_A3" device=""/>
-<part name="ART2" library="Custom_Eagle_KD" deviceset="ART_SN_LABEL" device="-08X24"/>
+<part name="SHEETINFO1" library="Custom_Eagle_KD" library_urn="urn:adsk.eagle:library:21708656" deviceset="ART_SHEET_INFO_1-16" device=""/>
+<part name="TEST_POINTS1" library="Custom_Eagle_KD" library_urn="urn:adsk.eagle:library:21708656" deviceset="ART_TEST_POINTS" device=""/>
+<part name="FIDUCIAL1" library="Custom_Eagle_KD" library_urn="urn:adsk.eagle:library:21708656" deviceset="FIDUCIAL" device="" package3d_urn="urn:adsk.eagle:package:21706180/1"/>
+<part name="FIDUCIAL2" library="Custom_Eagle_KD" library_urn="urn:adsk.eagle:library:21708656" deviceset="FIDUCIAL" device="" package3d_urn="urn:adsk.eagle:package:21706180/1"/>
+<part name="FIDUCIAL3" library="Custom_Eagle_KD" library_urn="urn:adsk.eagle:library:21708656" deviceset="FIDUCIAL" device="" package3d_urn="urn:adsk.eagle:package:21706180/1"/>
+<part name="FIDUCIAL4" library="Custom_Eagle_KD" library_urn="urn:adsk.eagle:library:21708656" deviceset="FIDUCIAL" device="" package3d_urn="urn:adsk.eagle:package:21706180/1"/>
+<part name="FIDUCIAL5" library="Custom_Eagle_KD" library_urn="urn:adsk.eagle:library:21708656" deviceset="FIDUCIAL" device="" package3d_urn="urn:adsk.eagle:package:21706180/1"/>
+<part name="FIDUCIAL6" library="Custom_Eagle_KD" library_urn="urn:adsk.eagle:library:21708656" deviceset="FIDUCIAL" device="" package3d_urn="urn:adsk.eagle:package:21706180/1"/>
+<part name="LOGO2" library="Custom_Eagle_KD" library_urn="urn:adsk.eagle:library:21708656" deviceset="ART_LOGO_TEXT_2.5MM" device="-SILK" package3d_urn="urn:adsk.eagle:package:21706313/1"/>
+<part name="LOGO3" library="Custom_Eagle_KD" library_urn="urn:adsk.eagle:library:21708656" deviceset="ART_LOGO_TEXT_2.5MM" device="-MASK" package3d_urn="urn:adsk.eagle:package:21706314/1"/>
+<part name="MTG5" library="Custom_Eagle_KD" library_urn="urn:adsk.eagle:library:21708656" deviceset="HOL_3.2/6.0_NP" device="-NOSILK" package3d_urn="urn:adsk.eagle:package:21706410/1" value="HOL_3.2/6.0_NP-NOSILK"/>
+<part name="MTG6" library="Custom_Eagle_KD" library_urn="urn:adsk.eagle:library:21708656" deviceset="HOL_3.2/6.0_NP" device="-NOSILK" package3d_urn="urn:adsk.eagle:package:21706410/1" value="HOL_3.2/6.0_NP-NOSILK"/>
+<part name="MTG4" library="Custom_Eagle_KD" library_urn="urn:adsk.eagle:library:21708656" deviceset="HOL_3.2/6.0_PTH" device="-3.2/6.0_PTH" package3d_urn="urn:adsk.eagle:package:21706149/2"/>
+<part name="GND18" library="Custom_Supply_Symbols_KD" library_urn="urn:adsk.eagle:library:21710300" deviceset="GND" device=""/>
+<part name="GND16" library="Custom_Supply_Symbols_KD" library_urn="urn:adsk.eagle:library:21710300" deviceset="GND" device=""/>
+<part name="REVINFO1" library="Custom_Eagle_KD" library_urn="urn:adsk.eagle:library:21708656" deviceset="ART_REVISION_HISTORY" device=""/>
+<part name="X1" library="Custom_Eagle_KD" library_urn="urn:adsk.eagle:library:21708656" deviceset="PAD_TEST_GROUND_HOOK" device="" package3d_urn="urn:adsk.eagle:package:21706157/2"/>
+<part name="MTG1" library="Custom_Eagle_KD" library_urn="urn:adsk.eagle:library:21708656" deviceset="HOL_2.2/4.2_NP" device="" package3d_urn="urn:adsk.eagle:package:21706303/1"/>
+<part name="MTG2" library="Custom_Eagle_KD" library_urn="urn:adsk.eagle:library:21708656" deviceset="HOL_2.2/4.2_NP" device="" package3d_urn="urn:adsk.eagle:package:21706303/1"/>
+<part name="MTG3" library="Custom_Eagle_KD" library_urn="urn:adsk.eagle:library:21708656" deviceset="HOL_2.2/4.2_NP" device="" package3d_urn="urn:adsk.eagle:package:21706303/1"/>
+<part name="MTG7" library="Custom_Eagle_KD" library_urn="urn:adsk.eagle:library:21708656" deviceset="HOL_2.2/4.2_NP" device="" package3d_urn="urn:adsk.eagle:package:21706303/1"/>
+<part name="ART1" library="Custom_Eagle_KD" library_urn="urn:adsk.eagle:library:21708656" deviceset="ART_QC" device="" package3d_urn="urn:adsk.eagle:package:21706350/1"/>
+<part name="TP1" library="Custom_Eagle_KD" library_urn="urn:adsk.eagle:library:21708656" deviceset="PAD_TEST_POINT" device="-2.5MM" package3d_urn="urn:adsk.eagle:package:21706159/2"/>
+<part name="TP2" library="Custom_Eagle_KD" library_urn="urn:adsk.eagle:library:21708656" deviceset="PAD_TEST_POINT" device="-2.5MM" package3d_urn="urn:adsk.eagle:package:21706159/2"/>
+<part name="TP3" library="Custom_Eagle_KD" library_urn="urn:adsk.eagle:library:21708656" deviceset="PAD_TEST_POINT" device="-2.5MM" package3d_urn="urn:adsk.eagle:package:21706159/2"/>
+<part name="FRAME1" library="Custom_Eagle_KD" library_urn="urn:adsk.eagle:library:21708656" deviceset="ART_FRAME_A3" device=""/>
+<part name="FRAME2" library="Custom_Eagle_KD" library_urn="urn:adsk.eagle:library:21708656" deviceset="ART_FRAME_A3" device=""/>
+<part name="FRAME3" library="Custom_Eagle_KD" library_urn="urn:adsk.eagle:library:21708656" deviceset="ART_FRAME_A3" device=""/>
+<part name="FRAME4" library="Custom_Eagle_KD" library_urn="urn:adsk.eagle:library:21708656" deviceset="ART_FRAME_A3" device=""/>
+<part name="FRAME5" library="Custom_Eagle_KD" library_urn="urn:adsk.eagle:library:21708656" deviceset="ART_FRAME_A3" device=""/>
+<part name="FRAME6" library="Custom_Eagle_KD" library_urn="urn:adsk.eagle:library:21708656" deviceset="ART_FRAME_A3" device=""/>
+<part name="FRAME7" library="Custom_Eagle_KD" library_urn="urn:adsk.eagle:library:21708656" deviceset="ART_FRAME_A3" device=""/>
+<part name="FRAME8" library="Custom_Eagle_KD" library_urn="urn:adsk.eagle:library:21708656" deviceset="ART_FRAME_A3" device=""/>
+<part name="FRAME9" library="Custom_Eagle_KD" library_urn="urn:adsk.eagle:library:21708656" deviceset="ART_FRAME_A3" device=""/>
+<part name="FRAME10" library="Custom_Eagle_KD" library_urn="urn:adsk.eagle:library:21708656" deviceset="ART_FRAME_A3" device=""/>
+<part name="ART2" library="Custom_Eagle_KD" library_urn="urn:adsk.eagle:library:21708656" deviceset="ART_SN_LABEL" device="-08X24" package3d_urn="urn:adsk.eagle:package:21706442/1"/>
 </parts>
 <sheets>
@@
 which will not be processed correctly with this version.
 </note>
+<note version="8.2" severity="warning">
+Since Version 8.2, EAGLE supports online libraries. The ids
+of those online libraries will not be understood (or retained)
+with this version.
+</note>
+<note version="8.3" severity="warning">
+Since Version 8.3, EAGLE supports URNs for individual library
+assets (packages, symbols, and devices). The URNs of those assets
+will not be understood (or retained) with this version.
+</note>
+<note version="8.3" severity="warning">
+Since Version 8.3, EAGLE supports the association of 3D packages
+with devices in libraries, schematics, and board files. Those 3D
+packages will not be understood (or retained) with this version.
+</note>
 </compatibility>
