File: templates/4-layer/000044 XXX Rev 1.00.sch (EAGLE design)
At the start: 22 parts, among them X1 PAD_TEST_GROUND_HOOK

Commit message: Changed templates to managed libraries
Parts:
- MTG5, MTG6: value HOL_3.2/6.0_NP -> HOL_3.2/6.0_NP-NOSILK; device Custom_Eagle_KD:HOL_3.2/6.0_NP -> Custom_Eagle_KD:HOL_3.2/6.0_NP-NOSILK
Other:
- moved on the sheet: ART1, ART2, FIDUCIAL1, FIDUCIAL2, FIDUCIAL3, FIDUCIAL4, FIDUCIAL5, FIDUCIAL6, LAYER1, LOGO2, LOGO3, MTG1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
